File: EPS/EPS_Board/EPS_Board.kicad_pcb (KiCad board)
At the start: 2 copper layers, 100 x 100 mm, 10 parts, among them J1 Conn_02x02_Counter_Clockwise, J2 Conn_01x04_Female, J3 Conn_01x04_Female, J4 Conn_01x04_Female, J5 Conn_01x04_Female, J6 Conn_01x04_Female, U1 AZ1117-3.3, U2 AZ1117-3.3, U3 AZ1117-5.0, U4 AZ1117-5.0

Commit message: Added caps for the lin regs. also added a led for coolnessss.
Parts:
- added C1: CAP, Capacitors_SMD:C_0805_HandSoldering, F.Cu at (182.9, 106.7)
- added C2: CAP, Capacitors_SMD:C_0805_HandSoldering, B.Cu at (156.2, 105.4)
- added C3: CAP, Capacitors_SMD:C_0805_HandSoldering, F.Cu at (113.0, 92.7)
- added D1: LED, LEDs:LED_0805_HandSoldering, F.Cu at (174.0, 109.2)
- added R1: R, Resistors_SMD:R_0805_HandSoldering, F.Cu at (183.0, 109.2)
Routing:
- net GND: track 7.66 -> 27.9 mm, vias 2 -> 5
- net Net-(D1-Pad1): track 0.00 -> 6.27 mm
- net +3V3: track 44.8 -> 49.6 mm
- net +BATT: track 21.6 -> 24.5 mm
